File: lis2dh12/lis2dh12.sch (KiCad schematic (older format))
At the start: 16 parts, among them J1 Conn_01x04_Male, J2 Conn_01x06_Male, U1 BME680

Commit message: Added LIS2DH sensor
Parts:
- removed U1: BME680, Package_LGA:Bosch_LGA-8_3x3mm_P0.8mm_ClockwisePinNumbering, symbol Sensor:BME680
- added U1: LIS2DH, Package_LGA:LGA-14_2x2mm_P0.35mm_LayoutBorder3x4y, symbol Sensor_Motion:LIS2DH
Connections:
- wire segments 53 -> 63
Other:
- note added: "ST LIS2DH"
- note removed: "Bosch BME680"
- moved on the sheet: C1, C2, JP1, R3
